File: pcb/rgb.kicad_pcb (KiCad board)
At the start: 2 copper layers, 128 x 30 mm, 22 parts, among them J1 Conn_02x08_Odd_Even, J2 Conn_01x02, J3 Conn_01x02, P1 TTL_232R_3V3, U1 ESP-WROOM-32, U2 LM317EMP, U3 RASPI_SD, U4 TACTILE, U5 TACTILE, U6 MicroSD_SPI_CD

Commit message: pcb: fix value of V-REG, Add info about SD card sockets
Parts:
- U2: value LM317EMP -> REG1117
- U3: value RASPI_SD -> 412D02F
